File: Steering Wheel.kicad_pcb (KiCad board)
At the start: 2 copper layers, 66.8 x 60 mm, 63 parts, among them J1 Conn_01x06_Socket, J2 Screw_Terminal_01x02, J3 Screw_Terminal_01x05, J4 Screw_Terminal_01x02, J5 Conn_01x05_Socket, SW1 SW_Push, SW2 SW_Push, SW3 SW_Push, SW4 SW_Push, SW5 SW_Push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

Commit message: made in update
Parts:
- removed kibuzzard-694BB84E: G***, kibuzzard-694BB84E
- moved kibuzzard-69775305 3.77 mm to (61.9, 70.8)
- moved kibuzzard-6977589B 3.77 mm to (61.9, 87.8)
